Commit message: Full model integration, specified inertia

File: ker_description/urdf/ker2.urdf (robot description, URDF)
Before this commit: robot ker, 9 links, 8 joints
Links:
- added link femur_1, mass 0.00167; collision box size=0.022 0.025 0.076; visual box size=0.022 0.025 0.076
- added link femur_2, mass 0.00167; collision box size=0.022 0.025 0.076; visual box size=0.022 0.025 0.076
- added link humerus_1, mass 0.00167; collision box size=0.022 0.025 0.076; visual box size=0.022 0.025 0.076
- added link humerus_2, mass 0.00167; collision box size=0.022 0.025 0.076; visual box size=0.022 0.025 0.076
- added link radius_1, mass 1; collision box size=0.022 0.025 0.04958; visual box size=0.022 0.025 0.04958
- added link radius_2, mass 1; collision box size=0.022 0.025 0.04958; visual box size=0.022 0.025 0.04958
- added link tibula_1, mass 1; collision box size=0.022 0.025 0.04958; visual box size=0.022 0.025 0.04958
- added link tibula_2, mass 1; collision box size=0.022 0.025 0.04958; visual box size=0.022 0.025 0.04958
- link big_motor_1: mass 0.5 -> 0.1
- link big_motor_2: mass 0.5 -> 0.1
- link big_motor_3: mass 0.5 -> 0.1
- link big_motor_4: mass 0.5 -> 0.1
- link body: geometry collision mesh filename=package://ker_description/meshes/start4_1.stl scale=1 1 1; visual mesh filename=package://ker_description/meshes/start4_1.stl scale=1 1 1
- link motor_1: mass 0.5 -> 0.00167
- link motor_2: mass 0.5 -> 0.00167
- link motor_3: mass 0.5 -> 0.00167
- link motor_4: mass 0.5 -> 0.00167
Joints:
- added joint femur_1_joint: type revolute, parent motor_4, child femur_1, origin xyz=0 0 0 rpy=0 0 0, axis 0 1 0, limit lower=-3.15 upper=3.15 effort=3.0 velocity=0.5
- added joint femur_2_joint: type revolute, parent motor_3, child femur_2, origin xyz=0 0 0 rpy=0 0 0, axis 0 -1 0, limit lower=-3.15 upper=3.15 effort=3.0 velocity=0.5
- added joint humerus_1_joint: type revolute, parent motor_1, child humerus_1, origin xyz=0 0 0 rpy=0 0 0, axis 0 1 0, limit lower=-3.15 upper=3.15 effort=3.0 velocity=0.5
- added joint humerus_2_joint: type revolute, parent motor_2, child humerus_2, origin xyz=0 0 0 rpy=0 0 0, axis 0 -1 0, limit lower=-3.15 upper=3.15 effort=3.0 velocity=0.5
- added joint radius_1_joint: type revolute, parent humerus_1, child radius_1, origin xyz=0 0 -0.076 rpy=0 0 0, axis 0 1 0, limit lower=-3.15 upper=3.15 effort=3.0 velocity=0.5
- added joint radius_2_joint: type revolute, parent humerus_2, child radius_2, origin xyz=0 0 -0.076 rpy=0 0 0, axis 0 -1 0, limit lower=-3.15 upper=3.15 effort=3.0 velocity=0.5
- added joint tibula_1_joint: type revolute, parent femur_1, child tibula_1, origin xyz=0 0 -0.076 rpy=0 0 0, axis 0 1 0, limit lower=-3.15 upper=3.15 effort=3.0 velocity=0.5
- added joint tibula_2_joint: type revolute, parent femur_2, child tibula_2, origin xyz=0 0 -0.076 rpy=0 0 0, axis 0 -1 0, limit lower=-3.15 upper=3.15 effort=3.0 velocity=0.5
- joint big_motor_1_joint: origin xyz=0.0745 0.0725 -0.011 rpy=0 0 0 -> xyz=0.049 0.0345 -0.0095 rpy=0 0 0
- joint big_motor_2_joint: origin xyz=0.0745 -0.0725 -0.011 rpy=0 0 0 -> xyz=0.049 -0.0345 -0.011 rpy=0 0 0
- joint big_motor_3_joint: origin xyz=-0.0745 -0.0725 -0.011 rpy=0 0 0 -> xyz=-0.049 -0.0345 -0.011 rpy=0 0 0
- joint big_motor_4_joint: origin xyz=-0.0745 0.0725 -0.011 rpy=0 0 0 -> xyz=-0.049 0.0345 -0.011 rpy=0 0 0
- joint motor_1_joint: limit lower=0.0 upper=3.15 effort=3.0 velocity=3.0 -> lower=-3.15 upper=3.15 effort=3.0 velocity=0.5
- joint motor_2_joint: limit lower=0.0 upper=3.15 effort=3.0 velocity=3.0 -> lower=-3.15 upper=3.15 effort=3.0 velocity=0.5
- joint motor_3_joint: limit lower=0.0 upper=3.15 effort=3.0 velocity=3.0 -> lower=-3.15 upper=3.15 effort=3.0 velocity=0.5
- joint motor_4_joint: limit lower=0.0 upper=3.15 effort=3.0 velocity=3.0 -> lower=-3.15 upper=3.15 effort=3.0 velocity=0.5
