Commit message: v0.02 - enabled ros_control

File: ker_description/robots/ker2.urdf.xacro (robot description, xacro)
@@ -58,5 +58,5 @@
             <axis xyz="${axis}"/>
             <dynamics damping="0.1" friction="0.1"/>
-            <limit effort="3.0" velocity="3.0" lower="0.0" upper="0.0"/>
+            <limit effort="3.0" velocity="3.0" lower="0.0" upper="3.15"/>
         </joint>
     </xacro:macro>
@@ -202,4 +202,5 @@
           <geometry>
             <box size = "${bodylen} ${bodywidth} ${bodyheight}"/>
+            <!--<mesh filename="package://ker_description/meshes/bucket_komp.STL" scale="0.001 0.001 0.001"/-->
           </geometry>
         </visual>

Commit message: v0.03 - sinusoidal joint movement code for low level walking

File: ker_description/robots/ker2.urdf.xacro (robot description, xacro)
@@ -22,4 +22,10 @@
     <xacro:property name="tibulalen" value="0.022" />
     <xacro:property name="tibulaheight" value="0.08" />
+   <physics type="ode" update_rate="100">
+     <gravity xyz="0 0 -9.81"/>
+         <ode>
+           <solver type="world" dt="0.01" iters="100" sor="1.3"/>
+         </ode>
+    </physics>
     <!--TRANSMISSION-->
     <xacro:macro name="ker_transmission" params="joint_name">
@@ -58,5 +64,5 @@
             <axis xyz="${axis}"/>
             <dynamics damping="0.1" friction="0.1"/>
-            <limit effort="3.0" velocity="3.0" lower="0.0" upper="3.15"/>
+            <limit effort="3.0" velocity="0.5" lower="-3.15" upper="3.15"/>
         </joint>
     </xacro:macro>
@@ -70,7 +76,4 @@
             </geometry>
             <origin xyz="0 0 0" rpy="0 0 0"/>
-            <material name="blue">
-                <color rgba="0 0 .8 1"/>
-            </material>
         </visual>
         <collision>
@@ -166,4 +169,9 @@
         </visual>
     </link>
+    <gazebo reference="${name}">
+      <mu1>1000</mu1>
+      <mu2>1000</mu2>
+      <material>Gazebo/Black</material>
+    </gazebo>
     <xacro:insert_block name="type" />
     <xacro:ker_transmission joint_name="${name}_joint" />
@@ -186,4 +194,8 @@
         </visual>
     </link>
+    <gazebo reference="${name}">
+      <mu1>1000</mu1>
+      <mu2>1000</mu2>
+    </gazebo>
     <xacro:insert_block name="type" />
     <xacro:ker_transmission joint_name="${name}_joint" />

Commit message: v0.06 - adapted model to new design, kinematics in Matlab

File: ker_description/robots/ker2.urdf.xacro (robot description, xacro)
@@ -18,8 +18,8 @@
     <xacro:property name="radiuswidth" value="0.025" />
     <xacro:property name="radiuslen" value="0.022" />
-    <xacro:property name="radiusheight" value="0.08" />
+    <xacro:property name="radiusheight" value="0.04958" />
     <xacro:property name="tibulawidth" value="0.025" />
     <xacro:property name="tibulalen" value="0.022" />
-    <xacro:property name="tibulaheight" value="0.08" />
+    <xacro:property name="tibulaheight" value="0.04958" />
    <physics type="ode" update_rate="100">
      <gravity xyz="0 0 -9.81"/>
@@ -44,7 +44,25 @@
         <inertial>
                 <mass value="${mass}" />
-                <inertia ixx="1.0" ixy="0.0" ixz="0.0"
-                     iyy="1.0" iyz="0.0"
-                     izz="1.0" />
+                <inertia ixx="0.001" ixy="0.0" ixz="0.0"
+                     iyy="0.001" iyz="0.0"
+                     izz="0.001" />
+        </inertial>
+    </xacro:macro>
+    <!--DYNAMIXEL INERTIAL PARAMETERS-->
+    <xacro:macro name="dynamixel_inertial" params="mass">
+        <inertial>
+                <mass value="0.00167" />
+                <inertia ixx="${0.08333333*motorwidth^2 + 0.08333333*motorheight^2}" ixy="0.0" ixz="0.0"
+                     iyy="${0.08333333*motorlen^2 + 0.08333333*motorheight^2}" iyz="0.0"
+                     izz="${0.08333333*motorlen^2 + 0.08333333*motorwidth^2}" />
+        </inertial>
+    </xacro:macro>
+    <!--HUMERUS AND FEMUR INERTIAL PARAMETERS-->
+    <xacro:macro name="humerus_femur_inertial" params="mass">
+        <inertial>
+                <mass value="0.00167" />
+                <inertia ixx="${0.08333333*humeruswidth^2 + 0.08333333*humerusheight^2}" ixy="0.0" ixz="0.0"
+                     iyy="${0.08333333*humeruslen^2 + 0.08333333*humerusheight^2}" iyz="0.0"
+                     izz="${0.08333333*humeruslen^2 + 0.08333333*humeruswidth^2}" />
         </inertial>
     </xacro:macro>
@@ -70,10 +88,10 @@
     <xacro:macro name="bigmotor" params="name pname origin">
     <link name="${name}">
-        <xacro:default_inertial mass="0.5"/>
+        <xacro:default_inertial mass="0.1"/>
         <visual>
             <geometry>
               <box size="${bigmotorlen} ${bigmotorwidth} ${bigmotorheight}"/>
             </geometry>
-            <origin xyz="0 0 0" rpy="0 0 0"/>
+            <origin xyz="0 0 0" rpy="${3.1415/2} 0 0"/>
         </visual>
         <collision>
@@ -93,5 +111,5 @@
     <xacro:macro name="motor" params="name *type">
     <link name="${name}">
-        <xacro:default_inertial mass="0.5"/>
+        <xacro:dynamixel_inertial mass="0.1"/>
         <visual>
             <geometry>
@@ -115,5 +133,5 @@
     <xacro:macro name="humerus" params="name *type">
     <link name="${name}">
-        <xacro:default_inertial mass="2"/>
+        <xacro:humerus_femur_inertial mass="1"/>
         <collision>
           <origin xyz="0 0 ${-motorheight/2-humerusheight/2}" rpy="0 0 0"/>
@@ -135,5 +153,5 @@
     <xacro:macro name="femur" params="name *type">
     <link name="${name}">
-        <xacro:default_inertial mass="2"/>
+        <xacro:humerus_femur_inertial mass="1"/>
         <collision>
           <origin xyz="0 0 ${-motorheight/2-femurheight/2}" rpy="0 0 0"/>
@@ -155,5 +173,5 @@
     <xacro:macro name="radius" params="name *type">
     <link name="${name}">
-        <xacro:default_inertial mass="2"/>
+        <xacro:default_inertial mass="1"/>
         <collision>
           <origin xyz="0 0 ${-motorheight/2-femurheight/2}" rpy="0 0 0"/>
@@ -166,29 +184,4 @@
           <geometry>
             <box size = "${radiuslen} ${radiuswidth} ${radiusheight}"/>
-          </geometry>
-        </visual>
-    </link>
-    <gazebo reference="${name}">
-      <mu1>1000</mu1>
-      <mu2>1000</mu2>
-      <material>Gazebo/Black</material>
-    </gazebo>
-    <xacro:insert_block name="type" />
-    <xacro:ker_transmission joint_name="${name}_joint" />
-    </xacro:macro>
-    <!--TIBULA-->
-    <xacro:macro name="tibula" params="name *type">
-    <link name="${name}">
-        <xacro:default_inertial mass="2"/>
-        <collision>
-          <origin xyz="0 0 ${-motorheight/2-tibulaheight/2}" rpy="0 0 0"/>
-          <geometry>
-            <box size="${tibulalen} ${tibulawidth} ${tibulaheight}"/>
-          </geometry>
-        </collision>
-        <visual>
-          <origin xyz="0 0 ${-motorheight/2-tibulaheight/2}" rpy="0 0 0"/>
-          <geometry>
-            <box size = "${tibulalen} ${tibulawidth} ${tibulaheight}"/>
           </geometry>
         </visual>
@@ -201,4 +194,28 @@
     <xacro:ker_transmission joint_name="${name}_joint" />
     </xacro:macro>
+    <!--TIBULA-->
+    <xacro:macro name="tibula" params="name *type">
+    <link name="${name}">
+        <xacro:default_inertial mass="1"/>
+        <collision>
+          <origin xyz="0 0 ${-motorheight/2-tibulaheight/2}" rpy="0 0 0"/>
+          <geometry>
+            <box size="${tibulalen} ${tibulawidth} ${tibulaheight}"/>
+          </geometry>
+        </collision>
+        <visual>
+          <origin xyz="0 0 ${-motorheight/2-tibulaheight/2}" rpy="0 0 0"/>
+          <geometry>
+            <box size = "${tibulalen} ${tibulawidth} ${tibulaheight}"/>
+          </geometry>
+        </visual>
+    </link>
+    <gazebo reference="${name}">
+      <mu1>1000</mu1>
+      <mu2>1000</mu2>
+    </gazebo>
+    <xacro:insert_block name="type" />
+    <xacro:ker_transmission joint_name="${name}_joint" />
+    </xacro:macro>
     <!--BODY-->
     <link name="body">
@@ -213,14 +230,14 @@
           <origin xyz="0 0 0.0" rpy="0 0 0"/>
           <geometry>
-            <box size = "${bodylen} ${bodywidth} ${bodyheight}"/>
-            <!--<mesh filename="package://ker_description/meshes/bucket_komp.STL" scale="0.001 0.001 0.001"/-->
+            <!--box size = "${bodylen} ${bodywidth} ${bodyheight}"/-->
+            <mesh filename="package://ker_description/meshes/start4_1.stl" scale="1 1 1"/>
           </geometry>
         </visual>
     </link>
     <!--EXECUTE MACROS-->
-    <xacro:bigmotor name="big_motor_1" pname="body" origin="${bodylen/2-bigmotorlen/2} ${bodywidth/2+bigmotorwidth/2} ${-bigmotorheight/2+bodyheight/2}" />
-    <xacro:bigmotor name="big_motor_2" pname="body" origin="${bodylen/2-bigmotorlen/2} ${-bodywidth/2-bigmotorwidth/2} ${-bigmotorheight/2+bodyheight/2}" />
-    <xacro:bigmotor name="big_motor_3" pname="body" origin="${-bodylen/2+bigmotorlen/2} ${-bodywidth/2-bigmotorwidth/2} ${-bigmotorheight/2+bodyheight/2}" />
-    <xacro:bigmotor name="big_motor_4" pname="body" origin="${-bodylen/2+bigmotorlen/2} ${bodywidth/2+bigmotorwidth/2} ${-bigmotorheight/2+bodyheight/2}" />
+    <xacro:bigmotor name="big_motor_1" pname="body" origin="${bodylen/2-bigmotorlen} ${bodywidth/2-bigmotorlen/2} ${-bigmotorwidth+bodyheight/2}" />
+    <xacro:bigmotor name="big_motor_2" pname="body" origin="${bodylen/2-bigmotorlen} ${-bodywidth/2+bigmotorlen/2} ${-bigmotorheight/2+bodyheight/2}" />
+    <xacro:bigmotor name="big_motor_3" pname="body" origin="${-bodylen/2+bigmotorlen} ${-bodywidth/2+bigmotorlen/2} ${-bigmotorheight/2+bodyheight/2}" />
+    <xacro:bigmotor name="big_motor_4" pname="body" origin="${-bodylen/2+bigmotorlen} ${bodywidth/2-bigmotorlen/2} ${-bigmotorheight/2+bodyheight/2}" />
     <xacro:motor name="motor_1">
         <xacro:revolute name="motor_1" pname="big_motor_1" origin="${bigmotorlen/2+motorlen/2} 0 0" axis="1 0 0"/>
@@ -251,5 +268,5 @@
         <xacro:revolute name="femur_1" pname="motor_4" origin="0 0 0" axis="0 1 0"/>
     </xacro:femur>
-    <xacro:motor name="motor_1b">
+    <!--xacro:motor name="motor_1b">
         <xacro:fixed name="motor_1b" pname="humerus_1" origin="0 0 -${humerusheight}" />
     </xacro:motor>
@@ -262,16 +279,16 @@
     <xacro:motor name="motor_4b">
         <xacro:fixed name="motor_4b" pname="femur_1" origin="0 0 -${femurheight}" />
-    </xacro:motor>
-        <xacro:radius name="radius_1" >
-        <xacro:revolute name="radius_1" pname="motor_1b" origin="0 0 0" axis="0 1 0"/>
+    </xacro:motor-->
+    <xacro:radius name="radius_1" >
+        <xacro:revolute name="radius_1" pname="humerus_1" origin="0 0 -${humerusheight}" axis="0 1 0"/>
     </xacro:radius>
     <xacro:radius name="radius_2" >
-        <xacro:revolute name="radius_2" pname="motor_2b" origin="0 0 0" axis="0 -1 0"/>
+        <xacro:revolute name="radius_2" pname="humerus_2" origin="0 0 -${humerusheight}" axis="0 -1 0"/>
     </xacro:radius>
     <xacro:tibula name="tibula_2" >
-        <xacro:revolute name="tibula_2" pname="motor_3b" origin="0 0 0" axis="0 -1 0"/>
+        <xacro:revolute name="tibula_2" pname="femur_2" origin="0 0 -${femurheight}" axis="0 -1 0"/>
     </xacro:tibula>
     <xacro:tibula name="tibula_1" >
-        <xacro:revolute name="tibula_1" pname="motor_4b" origin="0 0 0" axis="0 1 0"/>
+        <xacro:revolute name="tibula_1" pname="femur_1" origin="0 0 -${femurheight}" axis="0 1 0"/>
     </xacro:tibula>
     <gazebo>

Commit message: minor update to physics, ball contact model

File: ker_description/robots/ker2.urdf.xacro (robot description, xacro)
@@ -35,5 +35,5 @@
 	</xacro:macro>
     <!--BODY INERTIAL PARAMETERS-->
-    <xacro:macro name="default_inertial" params="mass">
+    <xacro:macro name="body_inertial">
         <inertial>
                 <origin rpy="0 0 0" xyz="0 0 0"/>
@@ -45,5 +45,5 @@
     </xacro:macro>
     <!--SHOULDER INERTIAL PARAMETERS-->
-    <xacro:macro name="dynamixel_inertial" params="mass">
+    <xacro:macro name="shoulder_inertial">
         <inertial>
                 <mass value="0.0082825" />
@@ -66,5 +66,5 @@
     <xacro:macro name="humerus_femur_inertial" params="mass">
         <inertial>
-                <origin rpy="0 0 0" xyz="0 0 ${-motorheight/2-humerusheight/2}"/>
+                <origin rpy="0 0 0" xyz="0 0 ${-humerusheight/2}"/>
                 <mass value="0.03619760" />
                 <inertia ixx="${1000*0.00000002198}" ixy="0.0" ixz="${1000*0.00000000004}"
@@ -76,5 +76,5 @@
     <xacro:macro name="radius_tibula_inertial" params="mass">
         <inertial>
-                <origin rpy="0 0 0" xyz="0 0 ${-humerusheight/2-radiusheight/2}"/>
+                <origin rpy="0 0 0" xyz="0 0 ${-humerusheight/2-radiusheight/2 + 0.037}"/>
                 <mass value="0.00992447" />
                 <inertia ixx="${0.00000000269*1000}" ixy="0.0" ixz="0.0"
@@ -97,41 +97,12 @@
             <origin xyz="${origin}" rpy="0 0 0"/>
             <axis xyz="${axis}"/>
-            <dynamics damping="0.1" friction="0.1"/>
-            <limit effort="3.0" velocity="0.5" lower="-3.15" upper="3.15"/>
+            <dynamics damping="0.0"/>
+            <limit effort="1.5" velocity="0.5" lower="-3.15" upper="3.15"/>
         </joint>
     </xacro:macro>
-    <!--MOTOR (CORONA)-->
-    <xacro:macro name="bigmotor" params="name pname origin">
-    <link name="${name}">
-        <inertial>
-                <origin rpy="0 0 0" xyz="${origin}"/>
-                <mass value="${2*0.000167}" />
-                <inertia ixx="${200*0.0167*0.08333333*bigmotorwidth^2 + 200*0.0167*0.08333333*bigmotorheight^2}" ixy="0.0" ixz="0.0"
-                     iyy="${200*0.0167*0.08333333*bigmotorlen^2 + 200*0.0167*0.08333333*bigmotorheight^2}" iyz="0.0"
-                     izz="${200*0.0167*0.08333333*bigmotorlen^2 + 200*0.0167*0.08333333*bigmotorwidth^2}" />
-        </inertial>
-        <visual>
-            <geometry>
-              <box size="${bigmotorlen} ${bigmotorwidth} ${bigmotorheight}"/>
-            </geometry>
-            <origin xyz="0 0 0" rpy="${3.1415/2} 0 0"/>
-        </visual>
-        <collision>
-            <geometry>
-              <box size="${bigmotorlen} ${bigmotorwidth} ${bigmotorheight}"/>
-            </geometry>
-            <origin xyz="0 0 0" rpy="${3.1415/2} 0 0"/>
-        </collision>
-    </link>
-    <joint name="${name}_joint" type="fixed">
-        <parent link="${pname}"/>
-        <child link="${name}"/>
-        <origin xyz="${origin}" rpy="0 0 0"/>
-    </joint>
-    </xacro:macro>
-    <!--MOTOR (DYNAMIXEL)-->
+    <!--SHOULDER-->
     <xacro:macro name="motor" params="name *type">
     <link name="${name}">
-        <xacro:dynamixel_inertial mass="0.1"/>
+        <xacro:shoulder_inertial/>
         <visual>
             <geometry>
@@ -159,5 +130,5 @@
         <xacro:humerus_femur_inertial mass="1"/>
         <collision>
-          <origin xyz="0 0 ${-motorheight/2-humerusheight/2 + 0.018}" rpy="0 0 0"/>
+          <origin xyz="0 0 ${-motorheight/2-humerusheight/2 +0.018 }" rpy="0 0 0"/>
           <geometry>
             <!--box size="${humeruslen} ${humeruswidth} ${humerusheight}"/-->
@@ -166,5 +137,5 @@
         </collision>
         <visual>
-          <origin xyz="0 0 ${-motorheight/2-humerusheight/2 + 0.018}" rpy="0 0 0"/>
+          <origin xyz="0 0 ${-motorheight/2-humerusheight/2 +0.018 }" rpy="0 0 0"/>
           <geometry>
             <!--box size = "${humeruslen} ${humeruswidth} ${humerusheight}"/-->
@@ -181,5 +152,5 @@
         <xacro:humerus_femur_inertial mass="1"/>
         <collision>
-          <origin xyz="0 0 ${-motorheight/2-femurheight/2 + 0.018}" rpy="0 0 0"/>
+          <origin xyz="0 0 ${-motorheight/2-femurheight/2 +0.018}" rpy="0 0 0"/>
           <geometry>
             <!--box size="${femurlen} ${femurwidth} ${femurheight}"/-->
@@ -188,5 +159,5 @@
         </collision>
         <visual>
-          <origin xyz="0 0 ${-motorheight/2-femurheight/2 + 0.018}" rpy="0 0 0"/>
+          <origin xyz="0 0 ${-motorheight/2-femurheight/2+0.018 }" rpy="0 0 0"/>
           <geometry>
             <mesh filename="package://ker_description/meshes/humerus.stl" scale="1 1 1"/>
@@ -203,8 +174,9 @@
         <xacro:radius_tibula_inertial mass="1"/>
         <collision>
-          <origin xyz="0 0 ${-motorheight/2-radiusheight/2 + 0.037}" rpy="0 0 0"/>
+          <origin xyz="0 0 ${-motorheight/2-radiusheight/2 +0.009}" rpy="0 0 0"/>
           <geometry>
             <!--box size="${radiuslen} ${radiuswidth} ${radiusheight}"/-->
-            <mesh filename="package://ker_description/meshes/radius.stl" scale="1 1 1"/>
+            <!--mesh filename="package://ker_description/meshes/radius.stl" scale="1 1 1"/-->
+            <sphere radius="0.01"/>
           </geometry>
         </collision>
@@ -218,6 +190,9 @@
     </link>
     <gazebo reference="${name}">
-      <mu1>1000</mu1>
-      <mu2>1000</mu2>
+      <minDepth>0.001</minDepth>
+      <maxContacts>1</maxContacts>
+      <fdir1>1 1 1</fdir1>
+      <mu1>1.0</mu1>
+      <mu2>100.0</mu2>
     </gazebo>
     <xacro:insert_block name="type" />
@@ -229,8 +204,9 @@
         <xacro:radius_tibula_inertial mass="1"/>
         <collision>
-          <origin xyz="0 0 ${-motorheight/2-tibulaheight/2 + 0.037}" rpy="0 0 0"/>
+          <origin xyz="0 0 ${-motorheight/2-tibulaheight/2 +0.009}" rpy="0 0 0"/>
           <geometry>
             <!--box size="${tibulalen} ${tibulawidth} ${tibulaheight}"/-->
-            <mesh filename="package://ker_description/meshes/radius.stl" scale="1 1 1"/>
+            <sphere radius="0.01"/>
+            <!--mesh filename="package://ker_description/meshes/radius.stl" scale="1 1 1"/-->
           </geometry>
         </collision>
@@ -244,6 +220,9 @@
     </link>
     <gazebo reference="${name}">
-      <mu1>1000</mu1>
-      <mu2>1000</mu2>
+      <minDepth>0.001</minDepth>
+      <maxContacts>1</maxContacts>
+      <fdir1>1 1 1</fdir1>
+      <mu1>1.0</mu1>
+      <mu2>100.0</mu2>
     </gazebo>
     <xacro:insert_block name="type" />
@@ -252,5 +231,5 @@
     <!--BODY-->
     <link name="body">
-        <xacro:default_inertial mass="0.6"/>
+        <xacro:body_inertial/>
         <collision>
           <origin xyz="0 0 0.0" rpy="0 0 0"/>
@@ -267,23 +246,18 @@
         </visual>
     </link>
-    <!--EXECUTE MACROS-->
-    <!--xacro:bigmotor name="big_motor_1" pname="body" origin="${bodylen/2-bigmotorlen} ${bodywidth/2-bigmotorlen/2} ${-bigmotorwidth+bodyheight/2}" />
-    <xacro:bigmotor name="big_motor_2" pname="body" origin="${bodylen/2-bigmotorlen} ${-bodywidth/2+bigmotorlen/2} ${-bigmotorheight/2+bodyheight/2}" />
-    <xacro:bigmotor name="big_motor_3" pname="body" origin="${-bodylen/2+bigmotorlen} ${-bodywidth/2+bigmotorlen/2} ${-bigmotorheight/2+bodyheight/2}" />
-    <xacro:bigmotor name="big_motor_4" pname="body" origin="${-bodylen/2+bigmotorlen} ${bodywidth/2-bigmotorlen/2} ${-bigmotorheight/2+bodyheight/2}" /-->
     <xacro:motor name="motor_1">
-        <xacro:revolute name="motor_1" pname="body" origin="${bodylen/2-motorlen-0.01} ${bodywidth/2-bigmotorlen/2} ${-bigmotorwidth -0.005 +bodyheight/2}" axis="1 0 0"/>
+        <xacro:revolute name="motor_1" pname="body" origin="${bodylen/2-motorlen-0.01} ${bodywidth/2-bigmotorlen/2} ${-bigmotorwidth +bodyheight/2 -0.005}" axis="1 0 0"/>
     </xacro:motor>
     <xacro:ker_transmission joint_name="motor_1_joint" />
     <xacro:motor name="motor_2">
-        <xacro:revolute name="motor_2" pname="body" origin="${bodylen/2-motorlen-0.01} ${-bodywidth/2+bigmotorlen/2} ${-bigmotorwidth -0.005 +bodyheight/2}" axis="1 0 0"/>
+        <xacro:revolute name="motor_2" pname="body" origin="${bodylen/2-motorlen-0.01} ${-bodywidth/2+bigmotorlen/2} ${-bigmotorwidth +bodyheight/2 -0.005}" axis="1 0 0"/>
     </xacro:motor>
     <xacro:ker_transmission joint_name="motor_2_joint" />
     <xacro:motor name="motor_3">
-        <xacro:revolute name="motor_3" pname="body" origin="${-bodylen/2+motorlen+0.01} ${-bodywidth/2+bigmotorlen/2} ${-bigmotorwidth -0.005 +bodyheight/2}" axis="1 0 0"/>
+        <xacro:revolute name="motor_3" pname="body" origin="${-bodylen/2+bigmotorheight+motorlen+0.01} ${-bodywidth/2+bigmotorlen/2} ${-bigmotorwidth +bodyheight/2 -0.005}" axis="1 0 0"/>
     </xacro:motor>
     <xacro:ker_transmission joint_name="motor_3_joint" />
     <xacro:motor name="motor_4">
-        <xacro:revolute name="motor_4" pname="body" origin="${-bodylen/2+motorlen+0.01} ${bodywidth/2-bigmotorlen/2} ${-bigmotorwidth -0.005 +bodyheight/2}" axis="1 0 0"/>
+        <xacro:revolute name="motor_4" pname="body" origin="${-bodylen/2+bigmotorheight+motorlen+0.01} ${bodywidth/2-bigmotorlen/2} ${-bigmotorwidth +bodyheight/2 -0.005}" axis="1 0 0"/>
     </xacro:motor>
     <xacro:ker_transmission joint_name="motor_4_joint" />

Commit message: modified contact parameters, no more oscillations

File: ker_description/robots/ker2.urdf.xacro (robot description, xacro)
@@ -98,5 +98,5 @@
             <axis xyz="${axis}"/>
             <dynamics damping="0.0"/>
-            <limit effort="1.5" velocity="0.5" lower="-3.15" upper="3.15"/>
+            <limit effort="1.5" velocity="0.5" lower="-3.14" upper="3.14"/>
         </joint>
     </xacro:macro>
@@ -190,9 +190,11 @@
     </link>
     <gazebo reference="${name}">
-      <minDepth>0.001</minDepth>
-      <maxContacts>1</maxContacts>
-      <fdir1>1 1 1</fdir1>
-      <mu1>1.0</mu1>
-      <mu2>100.0</mu2>
+        <kp>1000000.0</kp>
+        <kd>100.0</kd>
+        <mu1>1.0</mu1>
+        <mu2>1.0</mu2>
+        <fdir1>1 0 0</fdir1>
+        <maxVel>1.0</maxVel>
+        <minDepth>0.0</minDepth>
     </gazebo>
     <xacro:insert_block name="type" />
@@ -220,9 +222,11 @@
     </link>
     <gazebo reference="${name}">
-      <minDepth>0.001</minDepth>
-      <maxContacts>1</maxContacts>
-      <fdir1>1 1 1</fdir1>
-      <mu1>1.0</mu1>
-      <mu2>100.0</mu2>
+        <kp>1000000.0</kp>
+        <kd>100.0</kd>
+        <mu1>1.0</mu1>
+        <mu2>1.0</mu2>
+        <fdir1>1 0 0</fdir1>
+        <maxVel>1.0</maxVel>
+        <minDepth>0.0</minDepth>
     </gazebo>
     <xacro:insert_block name="type" />
