Commit message: v0.11-added rviz visualization, simulation global frame ground truth

File: ker_description/robots/ker.urdf.xacro (robot description, xacro)
@@ -35,5 +35,5 @@
 	</xacro:macro>
     <!--BODY INERTIAL PARAMETERS-->
-    <xacro:macro name="default_inertial" params="mass">
+    <xacro:macro name="body_inertial">
         <inertial>
                 <origin rpy="0 0 0" xyz="0 0 0"/>
@@ -45,6 +45,7 @@
     </xacro:macro>
     <!--SHOULDER INERTIAL PARAMETERS-->
-    <xacro:macro name="dynamixel_inertial" params="mass">
-        <inertial>
+    <xacro:macro name="shoulder_inertial">
+        <inertial>
+                <origin rpy="0 0 0" xyz="0 0 ${-bigmotorwidth/2}"/>
                 <mass value="0.0082825" />
                 <inertia ixx="${1000*0.00000000163}" ixy="0.0" ixz="0.0"
@@ -66,5 +67,5 @@
     <xacro:macro name="humerus_femur_inertial" params="mass">
         <inertial>
-                <origin rpy="0 0 0" xyz="0 0 ${-motorheight/2-humerusheight/2}"/>
+                <origin rpy="0 0 0" xyz="0 0 ${-humerusheight/2 + 0.01}"/>
                 <mass value="0.03619760" />
                 <inertia ixx="${1000*0.00000002198}" ixy="0.0" ixz="${1000*0.00000000004}"
@@ -76,5 +77,5 @@
     <xacro:macro name="radius_tibula_inertial" params="mass">
         <inertial>
-                <origin rpy="0 0 0" xyz="0 0 ${-humerusheight/2-radiusheight/2}"/>
+                <origin rpy="0 0 0" xyz="0 0 ${-radiusheight/2 +0.01}"/>
                 <mass value="0.00992447" />
                 <inertia ixx="${0.00000000269*1000}" ixy="0.0" ixz="0.0"
@@ -97,41 +98,12 @@
             <origin xyz="${origin}" rpy="0 0 0"/>
             <axis xyz="${axis}"/>
-            <dynamics damping="0.1" friction="0.1"/>
-            <limit effort="3.0" velocity="0.5" lower="-3.15" upper="3.15"/>
+            <dynamics damping="0.0"/>
+            <limit effort="1.5" velocity="0.5" lower="-3.14" upper="3.14"/>
         </joint>
     </xacro:macro>
-    <!--MOTOR (CORONA)-->
-    <xacro:macro name="bigmotor" params="name pname origin">
-    <link name="${name}">
-        <inertial>
-                <origin rpy="0 0 0" xyz="${origin}"/>
-                <mass value="${2*0.000167}" />
-                <inertia ixx="${200*0.0167*0.08333333*bigmotorwidth^2 + 200*0.0167*0.08333333*bigmotorheight^2}" ixy="0.0" ixz="0.0"
-                     iyy="${200*0.0167*0.08333333*bigmotorlen^2 + 200*0.0167*0.08333333*bigmotorheight^2}" iyz="0.0"
-                     izz="${200*0.0167*0.08333333*bigmotorlen^2 + 200*0.0167*0.08333333*bigmotorwidth^2}" />
-        </inertial>
-        <visual>
-            <geometry>
-              <box size="${bigmotorlen} ${bigmotorwidth} ${bigmotorheight}"/>
-            </geometry>
-            <origin xyz="0 0 0" rpy="${3.1415/2} 0 0"/>
-        </visual>
-        <collision>
-            <geometry>
-              <box size="${bigmotorlen} ${bigmotorwidth} ${bigmotorheight}"/>
-            </geometry>
-            <origin xyz="0 0 0" rpy="${3.1415/2} 0 0"/>
-        </collision>
-    </link>
-    <joint name="${name}_joint" type="fixed">
-        <parent link="${pname}"/>
-        <child link="${name}"/>
-        <origin xyz="${origin}" rpy="0 0 0"/>
-    </joint>
-    </xacro:macro>
-    <!--MOTOR (DYNAMIXEL)-->
+    <!--SHOULDER-->
     <xacro:macro name="motor" params="name *type">
     <link name="${name}">
-        <xacro:dynamixel_inertial mass="0.1"/>
+        <xacro:shoulder_inertial/>
         <visual>
             <geometry>
@@ -139,14 +111,15 @@
               <mesh filename="package://ker_description/meshes/roll.STL" scale="1 1 1"/>
             </geometry>
-            <origin xyz="0 0 0" rpy="0 0 0"/>
-            <material name="blue">
-                <color rgba="0 0 .8 1"/>
+            <origin xyz="0 0 ${-bigmotorwidth/2}" rpy="0 0 0"/>
+            <material name="grey">
+                <color rgba=".2 .2 .2 1"/>
             </material>
         </visual>
         <collision>
             <geometry>
-              <box size="${motorlen} ${motorwidth} ${motorheight}"/>
+              <!--box size="${motorlen} ${motorwidth} ${motorheight}"/-->
+              <mesh filename="package://ker_description/meshes/roll.STL" scale="1 1 1"/>
             </geometry>
-            <origin xyz="0 0 0" rpy="0 0 0"/>
+            <origin xyz="0 0 ${-bigmotorwidth/2}" rpy="0 0 0"/>
         </collision>
     </link>
@@ -158,15 +131,19 @@
         <xacro:humerus_femur_inertial mass="1"/>
         <collision>
-          <origin xyz="0 0 ${-motorheight/2-humerusheight/2}" rpy="0 0 0"/>
-          <geometry>
-            <box size="${humeruslen} ${humeruswidth} ${humerusheight}"/>
-          </geometry>
-        </collision>
-        <visual>
-          <origin xyz="0 0 ${-motorheight/2-humerusheight/2}" rpy="0 0 0"/>
+          <origin xyz="0 0 ${-humerusheight/2 + 0.01}" rpy="0 0 0"/>
+          <geometry>
+            <!--box size="${humeruslen} ${humeruswidth} ${humerusheight}"/-->
+            <mesh filename="package://ker_description/meshes/humerus.stl" scale="1 1 1"/>
+          </geometry>
+        </collision>
+        <visual>
+          <origin xyz="0 0 ${-humerusheight/2 + 0.01}" rpy="0 0 0"/>
           <geometry>
             <!--box size = "${humeruslen} ${humeruswidth} ${humerusheight}"/-->
             <mesh filename="package://ker_description/meshes/humerus.stl" scale="1 1 1"/>
           </geometry>
+          <material name="grey">
+              <color rgba=".2 .2 .2 1"/>
+          </material>
         </visual>
     </link>
@@ -179,16 +156,20 @@
         <xacro:humerus_femur_inertial mass="1"/>
         <collision>
-          <origin xyz="0 0 ${-motorheight/2-femurheight/2}" rpy="0 0 0"/>
-          <geometry>
-            <box size="${femurlen} ${femurwidth} ${femurheight}"/>
-          </geometry>
-        </collision>
-        <visual>
-          <origin xyz="0 0 ${-motorheight/2-femurheight/2}" rpy="0 0 0"/>
+          <origin xyz="0 0 ${-femurheight/2 + 0.01}" rpy="0 0 0"/>
+          <geometry>
+            <!--box size="${femurlen} ${femurwidth} ${femurheight}"/-->
+            <mesh filename="package://ker_description/meshes/humerus.stl" scale="1 1 1"/>
+          </geometry>
+        </collision>
+        <visual>
+          <origin xyz="0 0 ${-femurheight/2 + 0.01}" rpy="0 0 0"/>
           <geometry>
             <mesh filename="package://ker_description/meshes/humerus.stl" scale="1 1 1"/>
             <!--box size = "${femurlen} ${femurwidth} ${femurheight}"/-->
           </geometry>
-        </visual>
+          <material name="grey">
+              <color rgba=".2 .2 .2 1"/>
+          </material>
+       </visual>
     </link>
     <xacro:insert_block name="type" />
@@ -200,21 +181,30 @@
         <xacro:radius_tibula_inertial mass="1"/>
         <collision>
-          <origin xyz="0 0 ${-motorheight/2-femurheight/2}" rpy="0 0 0"/>
+          <origin xyz="0 0 ${-radiusheight + 0.008}" rpy="0 0 0"/>
           <geometry>
             <!--box size="${radiuslen} ${radiuswidth} ${radiusheight}"/-->
-            <mesh filename="package://ker_description/meshes/radius.stl" scale="1 1 1"/>
-          </geometry>
-        </collision>
-        <visual>
-          <origin xyz="0 0 ${-motorheight/2-radiusheight/2}" rpy="0 0 0"/>
+            <!--mesh filename="package://ker_description/meshes/radius.stl" scale="1 1 1"/-->
+            <sphere radius="0.01"/>
+          </geometry>
+        </collision>
+        <visual>
+          <origin xyz="0 0 ${-radiusheight/2+0.01}" rpy="0 0 0"/>
           <geometry>
             <mesh filename="package://ker_description/meshes/radius.stl" scale="1 1 1"/>
             <!--box size = "${radiuslen} ${radiuswidth} ${radiusheight}"/-->
           </geometry>
+          <material name="grey">
+              <color rgba=".2 .2 .2 1"/>
+          </material>
         </visual>
     </link>
     <gazebo reference="${name}">
-      <mu1>1000</mu1>
-      <mu2>1000</mu2>
+        <kp>1000000.0</kp>
+        <kd>100.0</kd>
+        <mu1>1000.0</mu1>
+        <mu2>1000.0</mu2>
+        <fdir1>1 1 0</fdir1>
+        <maxVel>1.0</maxVel>
+        <minDepth>0.0</minDepth>
     </gazebo>
     <xacro:insert_block name="type" />
@@ -226,21 +216,30 @@
         <xacro:radius_tibula_inertial mass="1"/>
         <collision>
-          <origin xyz="0 0 ${-motorheight/2-tibulaheight/2}" rpy="0 0 0"/>
+          <origin xyz="0 0 ${-tibulaheight +0.008}" rpy="0 0 0"/>
           <geometry>
             <!--box size="${tibulalen} ${tibulawidth} ${tibulaheight}"/-->
-            <mesh filename="package://ker_description/meshes/radius.stl" scale="1 1 1"/>
-          </geometry>
-        </collision>
-        <visual>
-          <origin xyz="0 0 ${-motorheight/2-tibulaheight/2}" rpy="0 0 0"/>
+            <sphere radius="0.01"/>
+            <!--mesh filename="package://ker_description/meshes/radius.stl" scale="1 1 1"/-->
+          </geometry>
+        </collision>
+        <visual>
+          <origin xyz="0 0 ${-tibulaheight/2 + 0.01}" rpy="0 0 0"/>
           <geometry>
             <!--box size = "${tibulalen} ${tibulawidth} ${tibulaheight}"/-->
             <mesh filename="package://ker_description/meshes/radius.stl" scale="1 1 1"/>
           </geometry>
+          <material name="grey">
+              <color rgba=".2 .2 .2 1"/>
+          </material>
         </visual>
     </link>
     <gazebo reference="${name}">
-      <mu1>1000</mu1>
-      <mu2>1000</mu2>
+        <kp>1000000.0</kp>
+        <kd>100.0</kd>
+        <mu1>1000.0</mu1>
+        <mu2>1000.0</mu2>
+        <fdir1>1 1 0</fdir1>
+        <maxVel>1.0</maxVel>
+        <minDepth>0.0</minDepth>
     </gazebo>
     <xacro:insert_block name="type" />
@@ -249,5 +248,5 @@
     <!--BODY-->
     <link name="body">
-        <xacro:default_inertial mass="0.6"/>
+        <xacro:body_inertial/>
         <collision>
           <origin xyz="0 0 0.0" rpy="0 0 0"/>
@@ -262,50 +261,64 @@
             <mesh filename="package://ker_description/meshes/platforma.stl" scale="1 1 1"/>
           </geometry>
-        </visual>
-    </link>
-    <!--EXECUTE MACROS-->
-    <!--xacro:bigmotor name="big_motor_1" pname="body" origin="${bodylen/2-bigmotorlen} ${bodywidth/2-bigmotorlen/2} ${-bigmotorwidth+bodyheight/2}" />
-    <xacro:bigmotor name="big_motor_2" pname="body" origin="${bodylen/2-bigmotorlen} ${-bodywidth/2+bigmotorlen/2} ${-bigmotorheight/2+bodyheight/2}" />
-    <xacro:bigmotor name="big_motor_3" pname="body" origin="${-bodylen/2+bigmotorlen} ${-bodywidth/2+bigmotorlen/2} ${-bigmotorheight/2+bodyheight/2}" />
-    <xacro:bigmotor name="big_motor_4" pname="body" origin="${-bodylen/2+bigmotorlen} ${bodywidth/2-bigmotorlen/2} ${-bigmotorheight/2+bodyheight/2}" /-->
+          <material name="grey">
+              <color rgba=".2 .2 .2 1"/>
+          </material>
+        </visual>
+    </link>
+    <!--DUMMY-->
+    <link name="odom">
+        <collision>
+          <origin xyz="0 0 0" rpy="0 0 0"/>
+          <geometry>
+            <box size = "0 0 0"/>
+          </geometry>
+        </collision>
+        <visual>
+          <origin xyz="0 0 0" rpy="0 0 0"/>
+          <geometry>
+            <box size = "0 0 0"/>
+          </geometry>
+        </visual>
+    </link>
+    <xacro:fixed name="body" pname="odom" origin="0 0 0"/>
     <xacro:motor name="motor_1">
-        <xacro:revolute name="motor_1" pname="body" origin="${bodylen/2-motorlen-0.01} ${bodywidth/2-bigmotorlen/2} ${-bigmotorwidth -0.005 +bodyheight/2}" axis="1 0 0"/>
+        <xacro:revolute name="motor_1" pname="body" origin="${bodylen/2-motorlen-0.01} ${bodywidth/2-bigmotorlen/2} ${-bigmotorwidth +bodyheight/2 + 0.01}" axis="1 0 0"/>
     </xacro:motor>
     <xacro:ker_transmission joint_name="motor_1_joint" />
     <xacro:motor name="motor_2">
-        <xacro:revolute name="motor_2" pname="body" origin="${bodylen/2-motorlen-0.01} ${-bodywidth/2+bigmotorlen/2} ${-bigmotorwidth -0.005 +bodyheight/2}" axis="1 0 0"/>
+        <xacro:revolute name="motor_2" pname="body" origin="${bodylen/2-motorlen-0.01} ${-bodywidth/2+bigmotorlen/2} ${-bigmotorwidth +bodyheight/2 + 0.01}" axis="1 0 0"/>
     </xacro:motor>
     <xacro:ker_transmission joint_name="motor_2_joint" />
     <xacro:motor name="motor_3">
-        <xacro:revolute name="motor_3" pname="body" origin="${-bodylen/2+motorlen+0.01} ${-bodywidth/2+bigmotorlen/2} ${-bigmotorwidth -0.005 +bodyheight/2}" axis="1 0 0"/>
+        <xacro:revolute name="motor_3" pname="body" origin="${-bodylen/2+bigmotorheight+motorlen+0.01} ${-bodywidth/2+bigmotorlen/2} ${-bigmotorwidth +bodyheight/2 + 0.01}" axis="1 0 0"/>
     </xacro:motor>
     <xacro:ker_transmission joint_name="motor_3_joint" />
     <xacro:motor name="motor_4">
-        <xacro:revolute name="motor_4" pname="body" origin="${-bodylen/2+motorlen+0.01} ${bodywidth/2-bigmotorlen/2} ${-bigmotorwidth -0.005 +bodyheight/2}" axis="1 0 0"/>
+        <xacro:revolute name="motor_4" pname="body" origin="${-bodylen/2+bigmotorheight+motorlen+0.01} ${bodywidth/2-bigmotorlen/2} ${-bigmotorwidth +bodyheight/2 + 0.01}" axis="1 0 0"/>
     </xacro:motor>
     <xacro:ker_transmission joint_name="motor_4_joint" />
     <xacro:humerus name="humerus_1">
-        <xacro:revolute name="humerus_1" pname="motor_1" origin="0 0 0" axis="0 1 0"/>
+        <xacro:revolute name="humerus_1" pname="motor_1" origin="0 0 ${-motorheight + 0.02}" axis="0 1 0"/> <!--1 za krug oko osi, 1 za sniženu os ramena/-->
     </xacro:humerus>
     <xacro:humerus name="humerus_2">
-        <xacro:revolute name="humerus_2" pname="motor_2" origin="0 0 0" axis="0 -1 0"/>
+        <xacro:revolute name="humerus_2" pname="motor_2" origin="0 0 ${-motorheight + 0.02}" axis="0 -1 0"/>
     </xacro:humerus>
     <xacro:femur name="femur_2">
-        <xacro:revolute name="femur_2" pname="motor_3" origin="0 0 0" axis="0 -1 0"/>
+        <xacro:revolute name="femur_2" pname="motor_3" origin="0 0 ${-motorheight + 0.02}" axis="0 -1 0"/>
     </xacro:femur>
     <xacro:femur name="femur_1">
-        <xacro:revolute name="femur_1" pname="motor_4" origin="0 0 0" axis="0 1 0"/>
+        <xacro:revolute name="femur_1" pname="motor_4" origin="0 0 ${-motorheight + 0.02}" axis="0 1 0"/>
     </xacro:femur>
     <xacro:radius name="radius_1" >
-        <xacro:revolute name="radius_1" pname="humerus_1" origin="0 0 -${humerusheight}" axis="0 1 0"/>
+        <xacro:revolute name="radius_1" pname="humerus_1" origin="0 0 ${-humerusheight + 0.02}" axis="0 1 0"/>
     </xacro:radius>
     <xacro:radius name="radius_2" >
-        <xacro:revolute name="radius_2" pname="humerus_2" origin="0 0 -${humerusheight}" axis="0 -1 0"/>
+        <xacro:revolute name="radius_2" pname="humerus_2" origin="0 0 ${-humerusheight + 0.02}" axis="0 -1 0"/>
     </xacro:radius>
     <xacro:tibula name="tibula_2" >
-        <xacro:revolute name="tibula_2" pname="femur_2" origin="0 0 -${femurheight}" axis="0 -1 0"/>
+        <xacro:revolute name="tibula_2" pname="femur_2" origin="0 0 ${-femurheight + 0.02}" axis="0 -1 0"/>
     </xacro:tibula>
     <xacro:tibula name="tibula_1" >
-        <xacro:revolute name="tibula_1" pname="femur_1" origin="0 0 -${femurheight}" axis="0 1 0"/>
+        <xacro:revolute name="tibula_1" pname="femur_1" origin="0 0 ${-femurheight + 0.02}" axis="0 1 0"/>
     </xacro:tibula>
     <gazebo>

Commit message: v0.121-fixed urdf stupidity

File: ker_description/robots/ker.urdf.xacro (robot description, xacro)
@@ -18,8 +18,10 @@
     <xacro:property name="radiuswidth" value="0.025" />
     <xacro:property name="radiuslen" value="0.022" />
-    <xacro:property name="radiusheight" value="0.04958" />
+    <xacro:property name="radiusheight" value="0.05958" />
     <xacro:property name="tibulawidth" value="0.025" />
     <xacro:property name="tibulalen" value="0.022" />
-    <xacro:property name="tibulaheight" value="0.04958" />
+    <xacro:property name="tibulaheight" value="0.05958" />
+    <xacro:property name="bodytoaxislen" value="0.073" />
+    <xacro:property name="bodytoaxiswidth" value="0.036" />
     <!--TRANSMISSION-->
     <xacro:macro name="ker_transmission" params="joint_name">
@@ -189,7 +191,7 @@
         </collision>
         <visual>
-          <origin xyz="0 0 ${-radiusheight/2+0.01}" rpy="0 0 0"/>
-          <geometry>
-            <mesh filename="package://ker_description/meshes/radius.stl" scale="1 1 1"/>
+          <origin xyz="0 0 ${-radiusheight/2+0.0135}" rpy="0 0 0"/>
+          <geometry>
+            <mesh filename="package://ker_description/meshes/radius_3_dec.STL" scale="1 1 1"/>
             <!--box size = "${radiuslen} ${radiuswidth} ${radiusheight}"/-->
           </geometry>
@@ -224,8 +226,8 @@
         </collision>
         <visual>
-          <origin xyz="0 0 ${-tibulaheight/2 + 0.01}" rpy="0 0 0"/>
+          <origin xyz="0 0 ${-tibulaheight/2 + 0.0135}" rpy="0 0 0"/>
           <geometry>
             <!--box size = "${tibulalen} ${tibulawidth} ${tibulaheight}"/-->
-            <mesh filename="package://ker_description/meshes/radius.stl" scale="1 1 1"/>
+            <mesh filename="package://ker_description/meshes/radius_3_dec.STL" scale="1 1 1"/>
           </geometry>
           <material name="grey">
@@ -253,5 +255,5 @@
           <geometry>
             <!--box size = "${bodylen} ${bodywidth} ${bodyheight}"/-->
-            <mesh filename="package://ker_description/meshes/platforma.stl" scale="1 1 1"/>
+            <mesh filename="package://ker_description/meshes/platf_3_1.STL" scale="1 1 1"/>
           </geometry>
         </collision>
@@ -259,5 +261,5 @@
           <origin xyz="0 0 0.0" rpy="0 0 0"/>
           <geometry>
-            <mesh filename="package://ker_description/meshes/platforma.stl" scale="1 1 1"/>
+            <mesh filename="package://ker_description/meshes/platf_3_1.STL" scale="1 1 1"/>
           </geometry>
           <material name="grey">
@@ -283,17 +285,17 @@
     <xacro:fixed name="body" pname="odom" origin="0 0 0"/>
     <xacro:motor name="motor_1">
-        <xacro:revolute name="motor_1" pname="body" origin="${bodylen/2-motorlen-0.01} ${bodywidth/2-bigmotorlen/2} ${-bigmotorwidth +bodyheight/2 + 0.01}" axis="1 0 0"/>
+        <xacro:revolute name="motor_1" pname="body" origin="${bodytoaxislen} ${bodytoaxiswidth} ${-bigmotorwidth +bodyheight/2 + 0.01}" axis="1 0 0"/>
     </xacro:motor>
     <xacro:ker_transmission joint_name="motor_1_joint" />
     <xacro:motor name="motor_2">
-        <xacro:revolute name="motor_2" pname="body" origin="${bodylen/2-motorlen-0.01} ${-bodywidth/2+bigmotorlen/2} ${-bigmotorwidth +bodyheight/2 + 0.01}" axis="1 0 0"/>
+        <xacro:revolute name="motor_2" pname="body" origin="${bodytoaxislen} ${-bodytoaxiswidth} ${-bigmotorwidth +bodyheight/2 + 0.01}" axis="1 0 0"/>
     </xacro:motor>
     <xacro:ker_transmission joint_name="motor_2_joint" />
     <xacro:motor name="motor_3">
-        <xacro:revolute name="motor_3" pname="body" origin="${-bodylen/2+bigmotorheight+motorlen+0.01} ${-bodywidth/2+bigmotorlen/2} ${-bigmotorwidth +bodyheight/2 + 0.01}" axis="1 0 0"/>
+        <xacro:revolute name="motor_3" pname="body" origin="${-bodytoaxislen} ${-bodytoaxiswidth} ${-bigmotorwidth +bodyheight/2 + 0.01}" axis="1 0 0"/>
     </xacro:motor>
     <xacro:ker_transmission joint_name="motor_3_joint" />
     <xacro:motor name="motor_4">
-        <xacro:revolute name="motor_4" pname="body" origin="${-bodylen/2+bigmotorheight+motorlen+0.01} ${bodywidth/2-bigmotorlen/2} ${-bigmotorwidth +bodyheight/2 + 0.01}" axis="1 0 0"/>
+        <xacro:revolute name="motor_4" pname="body" origin="${-bodytoaxislen} ${bodytoaxiswidth} ${-bigmotorwidth +bodyheight/2 + 0.01}" axis="1 0 0"/>
     </xacro:motor>
     <xacro:ker_transmission joint_name="motor_4_joint" />
