Commit message: v0.13 Jacobian kinematics test-bench (still needs work), urdf optimization

File: ker_description/robots/ker.urdf.xacro (robot description, xacro)
@@ -1,4 +1,5 @@
 <?xml version='1.0'?>
   <robot xmlns:xacro="http://www.ros.org/wiki/xacro" name="ker">
+    <xacro:property name="pi" value="3.14159265359" />
     <xacro:property name="bodywidth" value=".12000000" />
     <xacro:property name="bodylen" value=".200000000" />
@@ -18,8 +19,8 @@
     <xacro:property name="radiuswidth" value="0.025" />
     <xacro:property name="radiuslen" value="0.022" />
-    <xacro:property name="radiusheight" value="0.05958" />
+    <xacro:property name="radiusheight" value="0.06856" />
     <xacro:property name="tibulawidth" value="0.025" />
     <xacro:property name="tibulalen" value="0.022" />
-    <xacro:property name="tibulaheight" value="0.05958" />
+    <xacro:property name="tibulaheight" value="0.06856" />
     <xacro:property name="bodytoaxislen" value="0.073" />
     <xacro:property name="bodytoaxiswidth" value="0.036" />
@@ -94,12 +95,12 @@
         </joint>
     </xacro:macro>
-    <xacro:macro name="revolute" params="name pname origin axis">
+    <xacro:macro name="revolute" params="name pname origin rot axis">
         <joint name="${name}_joint" type="revolute">
             <parent link="${pname}"/>
             <child link="${name}"/>
-            <origin xyz="${origin}" rpy="0 0 0"/>
+            <origin xyz="${origin}" rpy="${rot}"/>
             <axis xyz="${axis}"/>
             <dynamics damping="0.0"/>
-            <limit effort="1.5" velocity="0.5" lower="-3.14" upper="3.14"/>
+            <limit effort="10" velocity="0.5" lower="-3.14" upper="3.14"/>
         </joint>
     </xacro:macro>
@@ -120,6 +121,6 @@
         <collision>
             <geometry>
-              <!--box size="${motorlen} ${motorwidth} ${motorheight}"/-->
-              <mesh filename="package://ker_description/meshes/roll.STL" scale="1 1 1"/>
+              <box size="${motorlen} ${motorwidth} ${motorheight}"/>
+              <!--mesh filename="package://ker_description/meshes/roll.STL" scale="1 1 1"/-->
             </geometry>
             <origin xyz="0 0 ${-bigmotorwidth/2}" rpy="0 0 0"/>
@@ -135,6 +136,6 @@
           <origin xyz="0 0 ${-humerusheight/2 + 0.01}" rpy="0 0 0"/>
           <geometry>
-            <!--box size="${humeruslen} ${humeruswidth} ${humerusheight}"/-->
-            <mesh filename="package://ker_description/meshes/humerus.stl" scale="1 1 1"/>
+            <box size="${humeruslen} ${humeruswidth} ${humerusheight}"/>
+            <!--mesh filename="package://ker_description/meshes/humerus.stl" scale="1 1 1"/-->
           </geometry>
         </collision>
@@ -160,6 +161,6 @@
           <origin xyz="0 0 ${-femurheight/2 + 0.01}" rpy="0 0 0"/>
           <geometry>
-            <!--box size="${femurlen} ${femurwidth} ${femurheight}"/-->
-            <mesh filename="package://ker_description/meshes/humerus.stl" scale="1 1 1"/>
+            <box size="${femurlen} ${femurwidth} ${femurheight}"/>
+            <!--mesh filename="package://ker_description/meshes/humerus.stl" scale="1 1 1"/-->
           </geometry>
         </collision>
@@ -183,13 +184,13 @@
         <xacro:radius_tibula_inertial mass="1"/>
         <collision>
-          <origin xyz="0 0 ${-radiusheight + 0.008}" rpy="0 0 0"/>
+          <origin xyz="0 0 ${-radiusheight/2 + 0.018}" rpy="0 0 0"/>
           <geometry>
             <!--box size="${radiuslen} ${radiuswidth} ${radiusheight}"/-->
-            <!--mesh filename="package://ker_description/meshes/radius.stl" scale="1 1 1"/-->
-            <sphere radius="0.01"/>
-          </geometry>
-        </collision>
-        <visual>
-          <origin xyz="0 0 ${-radiusheight/2+0.0135}" rpy="0 0 0"/>
+            <mesh filename="package://ker_description/meshes/radius_3_dec.STL" scale="1 1 1"/>
+            <!--sphere radius="0.001"/-->
+          </geometry>
+        </collision>
+        <visual>
+          <origin xyz="0 0 ${-radiusheight/2+0.018}" rpy="0 0 0"/>
           <geometry>
             <mesh filename="package://ker_description/meshes/radius_3_dec.STL" scale="1 1 1"/>
@@ -202,11 +203,11 @@
     </link>
     <gazebo reference="${name}">
-        <kp>1000000.0</kp>
-        <kd>100.0</kd>
-        <mu1>1000.0</mu1>
-        <mu2>1000.0</mu2>
-        <fdir1>1 1 0</fdir1>
-        <maxVel>1.0</maxVel>
-        <minDepth>0.0</minDepth>
+        <kp>100000.0</kp>
+        <kd>1.0</kd>
+        <mu1>100000.0</mu1>
+        <mu2>100000.0</mu2>
+        <fdir1>1 1 1</fdir1>
+        <maxVel>1.2</maxVel>
+        <minDepth>0.01</minDepth>
     </gazebo>
     <xacro:insert_block name="type" />
@@ -218,13 +219,13 @@
         <xacro:radius_tibula_inertial mass="1"/>
         <collision>
-          <origin xyz="0 0 ${-tibulaheight +0.008}" rpy="0 0 0"/>
+          <origin xyz="0 0 ${-tibulaheight/2 +0.018}" rpy="0 0 0"/>
           <geometry>
             <!--box size="${tibulalen} ${tibulawidth} ${tibulaheight}"/-->
-            <sphere radius="0.01"/>
-            <!--mesh filename="package://ker_description/meshes/radius.stl" scale="1 1 1"/-->
-          </geometry>
-        </collision>
-        <visual>
-          <origin xyz="0 0 ${-tibulaheight/2 + 0.0135}" rpy="0 0 0"/>
+            <!--sphere radius="0.001"/-->
+            <mesh filename="package://ker_description/meshes/radius_3_dec.STL" scale="1 1 1"/>
+          </geometry>
+        </collision>
+        <visual>
+          <origin xyz="0 0 ${-tibulaheight/2 + 0.018}" rpy="0 0 0"/>
           <geometry>
             <!--box size = "${tibulalen} ${tibulawidth} ${tibulaheight}"/-->
@@ -237,11 +238,11 @@
     </link>
     <gazebo reference="${name}">
-        <kp>1000000.0</kp>
-        <kd>100.0</kd>
-        <mu1>1000.0</mu1>
-        <mu2>1000.0</mu2>
-        <fdir1>1 1 0</fdir1>
-        <maxVel>1.0</maxVel>
-        <minDepth>0.0</minDepth>
+        <kp>100000.0</kp>
+        <kd>1.0</kd>
+        <mu1>100000.0</mu1>
+        <mu2>100000.0</mu2>
+        <fdir1>1 1 1</fdir1>
+        <maxVel>1.2</maxVel>
+        <minDepth>0.00</minDepth>
     </gazebo>
     <xacro:insert_block name="type" />
@@ -254,6 +255,6 @@
           <origin xyz="0 0 0.0" rpy="0 0 0"/>
           <geometry>
-            <!--box size = "${bodylen} ${bodywidth} ${bodyheight}"/-->
-            <mesh filename="package://ker_description/meshes/platf_3_1.STL" scale="1 1 1"/>
+            <box size = "${bodylen} ${bodywidth} ${bodyheight}"/>
+            <!--mesh filename="package://ker_description/meshes/platf_3_1.STL" scale="1 1 1"/-->
           </geometry>
         </collision>
@@ -285,42 +286,42 @@
     <xacro:fixed name="body" pname="odom" origin="0 0 0"/>
     <xacro:motor name="motor_1">
-        <xacro:revolute name="motor_1" pname="body" origin="${bodytoaxislen} ${bodytoaxiswidth} ${-bigmotorwidth +bodyheight/2 + 0.01}" axis="1 0 0"/>
+        <xacro:revolute name="motor_1" pname="body" origin="${bodytoaxislen} ${bodytoaxiswidth} ${-bigmotorwidth +bodyheight/2 + 0.01}" rot = "0 0 0" axis="1 0 0"/>
     </xacro:motor>
     <xacro:ker_transmission joint_name="motor_1_joint" />
     <xacro:motor name="motor_2">
-        <xacro:revolute name="motor_2" pname="body" origin="${bodytoaxislen} ${-bodytoaxiswidth} ${-bigmotorwidth +bodyheight/2 + 0.01}" axis="1 0 0"/>
+        <xacro:revolute name="motor_2" pname="body" origin="${bodytoaxislen} ${-bodytoaxiswidth} ${-bigmotorwidth +bodyheight/2 + 0.01}" rot = "0 0 0" axis="1 0 0"/>
     </xacro:motor>
     <xacro:ker_transmission joint_name="motor_2_joint" />
     <xacro:motor name="motor_3">
-        <xacro:revolute name="motor_3" pname="body" origin="${-bodytoaxislen} ${-bodytoaxiswidth} ${-bigmotorwidth +bodyheight/2 + 0.01}" axis="1 0 0"/>
+        <xacro:revolute name="motor_3" pname="body" origin="${-bodytoaxislen} ${-bodytoaxiswidth} ${-bigmotorwidth +bodyheight/2 + 0.01}" rot = "0 0 0" axis="1 0 0"/>
     </xacro:motor>
     <xacro:ker_transmission joint_name="motor_3_joint" />
     <xacro:motor name="motor_4">
-        <xacro:revolute name="motor_4" pname="body" origin="${-bodytoaxislen} ${bodytoaxiswidth} ${-bigmotorwidth +bodyheight/2 + 0.01}" axis="1 0 0"/>
+        <xacro:revolute name="motor_4" pname="body" origin="${-bodytoaxislen} ${bodytoaxiswidth} ${-bigmotorwidth +bodyheight/2 + 0.01}" rot = "0 0 0" axis="1 0 0"/>
     </xacro:motor>
     <xacro:ker_transmission joint_name="motor_4_joint" />
     <xacro:humerus name="humerus_1">
-        <xacro:revolute name="humerus_1" pname="motor_1" origin="0 0 ${-motorheight + 0.02}" axis="0 1 0"/> <!--1 za krug oko osi, 1 za sniženu os ramena/-->
+        <xacro:revolute name="humerus_1" pname="motor_1" origin="0 0 ${-motorheight + 0.02}" rot = "0 0 0" axis="0 1 0"/>
     </xacro:humerus>
     <xacro:humerus name="humerus_2">
-        <xacro:revolute name="humerus_2" pname="motor_2" origin="0 0 ${-motorheight + 0.02}" axis="0 -1 0"/>
+        <xacro:revolute name="humerus_2" pname="motor_2" origin="0 0 ${-motorheight + 0.02}" rot = "0 0 ${pi}" axis="0 -1 0"/>
     </xacro:humerus>
     <xacro:femur name="femur_2">
-        <xacro:revolute name="femur_2" pname="motor_3" origin="0 0 ${-motorheight + 0.02}" axis="0 -1 0"/>
+        <xacro:revolute name="femur_2" pname="motor_3" origin="0 0 ${-motorheight + 0.02}" rot = "0 0 ${pi}" axis="0 -1 0"/>
     </xacro:femur>
     <xacro:femur name="femur_1">
-        <xacro:revolute name="femur_1" pname="motor_4" origin="0 0 ${-motorheight + 0.02}" axis="0 1 0"/>
+        <xacro:revolute name="femur_1" pname="motor_4" origin="0 0 ${-motorheight + 0.02}" rot = "0 0 0" axis="0 1 0"/>
     </xacro:femur>
     <xacro:radius name="radius_1" >
-        <xacro:revolute name="radius_1" pname="humerus_1" origin="0 0 ${-humerusheight + 0.02}" axis="0 1 0"/>
+        <xacro:revolute name="radius_1" pname="humerus_1" origin="0 0 ${-humerusheight + 0.02}" rot = "0 0 0" axis="0 1 0"/>
     </xacro:radius>
     <xacro:radius name="radius_2" >
-        <xacro:revolute name="radius_2" pname="humerus_2" origin="0 0 ${-humerusheight + 0.02}" axis="0 -1 0"/>
+        <xacro:revolute name="radius_2" pname="humerus_2" origin="0 0 ${-humerusheight + 0.02}" rot = "0 0 0" axis="0 -1 0"/>
     </xacro:radius>
     <xacro:tibula name="tibula_2" >
-        <xacro:revolute name="tibula_2" pname="femur_2" origin="0 0 ${-femurheight + 0.02}" axis="0 -1 0"/>
+        <xacro:revolute name="tibula_2" pname="femur_2" origin="0 0 ${-femurheight + 0.02}" rot = "0 0 0" axis="0 -1 0"/>
     </xacro:tibula>
     <xacro:tibula name="tibula_1" >
-        <xacro:revolute name="tibula_1" pname="femur_1" origin="0 0 ${-femurheight + 0.02}" axis="0 1 0"/>
+        <xacro:revolute name="tibula_1" pname="femur_1" origin="0 0 ${-femurheight + 0.02}" rot = "0 0 0" axis="0 1 0"/>
     </xacro:tibula>
     <gazebo>
