Commit message: v0.21 - added constraints to IK | IK solutions filtered with closest criterion

File: ker_description/robots/ker_analytic.urdf.xacro (robot description, xacro)
@@ -38,5 +38,5 @@
         <type>transmission_interface/SimpleTransmission</type>
           <joint name="${joint_name}">
-            <hardwareInterface>EffortJointInterface</hardwareInterface>
+            <hardwareInterface>PositionJointInterface</hardwareInterface>
           </joint>
           <actuator name="${joint_name}_motor">
@@ -110,5 +110,5 @@
             <axis xyz="${axis}"/>
             <dynamics damping="0.002" friction="0.01"/>
-            <limit effort="0.4" velocity="0.5" lower="-3.14" upper="3.14"/>
+            <limit effort="0.4" velocity="10" lower="-3.14" upper="3.14"/>
         </joint>
     </xacro:macro>

Commit message: v0.25b-new tf stuff

File: ker_description/robots/ker_analytic.urdf.xacro (robot description, xacro)
@@ -110,5 +110,5 @@
             <axis xyz="${axis}"/>
             <dynamics damping="0.002" friction="0.01"/>
-            <limit effort="0.4" velocity="10" lower="-3.14" upper="3.14"/>
+            <limit effort="0.4" velocity="0.5" lower="-3.14" upper="3.14"/>
         </joint>
     </xacro:macro>
